File: RF.kicad_sch (KiCad schematic)
At the start: 12 parts, among them J1 Conn_Coaxial, J3 Conn_Coaxial, U4 ADG902BRMZ

Commit message: add initial pinouts and USB
Parts:
- renumbered C20 to C22, C24 to C23, C23 to C24, J1 to J2, L5 to L3, L3 to L4, L4 to L5, U4 to U6
Changed lines of the file:
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@@
 		(dnp no)
 		(fields_autoplaced yes)
-		(property "Reference" "L5"
+		(property "Reference" "L3"
 			(at 168.91 77.47 90)
 			(show_name no)
@@
 			(project "WINLAB-LP-Radio-Sensor-Hub"
 				(path "/0de7ee4a-bb98-4bc6-bb89-3afafc4b94b5/415caeb0-0f13-4c6e-8f8f-fa1df5ea5ac9"
-					(reference "L5")
+					(reference "L3")
 					(unit 1)
 				)
@@
 		(dnp no)
 		(fields_autoplaced yes)
-		(property "Reference" "J1"
+		(property "Reference" "J2"
 			(at 116.84 77.7631 0)
 			(show_name no)
@@
 			(project "WINLAB-LP-Radio-Sensor-Hub"
 				(path "/0de7ee4a-bb98-4bc6-bb89-3afafc4b94b5/415caeb0-0f13-4c6e-8f8f-fa1df5ea5ac9"
-					(reference "J1")
+					(reference "J2")
 					(unit 1)
 				)
@@
 		(dnp no)
 		(fields_autoplaced yes)
-		(property "Reference" "C23"
+		(property "Reference" "C24"
 			(at 194.31 69.8499 0)
 			(show_name no)
@@
 			(project "WINLAB-LP-Radio-Sensor-Hub"
 				(path "/0de7ee4a-bb98-4bc6-bb89-3afafc4b94b5/415caeb0-0f13-4c6e-8f8f-fa1df5ea5ac9"
-					(reference "C23")
+					(reference "C24")
 					(unit 1)
 				)
@@
 		(dnp no)
 		(fields_autoplaced yes)
-		(property "Reference" "C24"
+		(property "Reference" "C23"
 			(at 168.91 49.53 90)
 			(show_name no)
@@
 			(project "WINLAB-LP-Radio-Sensor-Hub"
 				(path "/0de7ee4a-bb98-4bc6-bb89-3afafc4b94b5/415caeb0-0f13-4c6e-8f8f-fa1df5ea5ac9"
-					(reference "C24")
+					(reference "C23")
 					(unit 1)
 				)
@@
 		(dnp no)
 		(fields_autoplaced yes)
-		(property "Reference" "C20"
+		(property "Reference" "C22"
 			(at 95.25 57.1499 0)
 			(show_name no)
@@
 			(project "WINLAB-LP-Radio-Sensor-Hub"
 				(path "/0de7ee4a-bb98-4bc6-bb89-3afafc4b94b5/415caeb0-0f13-4c6e-8f8f-fa1df5ea5ac9"
-					(reference "C20")
+					(reference "C22")
 					(unit 1)
 				)
@@
 		(dnp no)
 		(fields_autoplaced yes)
-		(property "Reference" "#PWR015"
+		(property "Reference" "#PWR020"
 			(at 91.44 58.42 0)
 			(hide yes)
@@
 			(project "WINLAB-LP-Radio-Sensor-Hub"
 				(path "/0de7ee4a-bb98-4bc6-bb89-3afafc4b94b5/415caeb0-0f13-4c6e-8f8f-fa1df5ea5ac9"
-					(reference "#PWR015")
+					(reference "#PWR020")
 					(unit 1)
 				)
@@
 		(dnp no)
 		(fields_autoplaced yes)
-		(property "Reference" "L4"
+		(property "Reference" "L5"
 			(at 199.39 62.23 90)
 			(show_name no)
@@
 			(project "WINLAB-LP-Radio-Sensor-Hub"
 				(path "/0de7ee4a-bb98-4bc6-bb89-3afafc4b94b5/415caeb0-0f13-4c6e-8f8f-fa1df5ea5ac9"
-					(reference "L4")
+					(reference "L5")
 					(unit 1)
 				)
@@
 		(dnp no)
 		(fields_autoplaced yes)
-		(property "Reference" "#PWR018"
+		(property "Reference" "#PWR019"
 			(at 85.09 102.87 0)
 			(hide yes)
@@
 			(project "WINLAB-LP-Radio-Sensor-Hub"
 				(path "/0de7ee4a-bb98-4bc6-bb89-3afafc4b94b5/415caeb0-0f13-4c6e-8f8f-fa1df5ea5ac9"
-					(reference "#PWR018")
+					(reference "#PWR019")
 					(unit 1)
 				)
@@
 		(dnp no)
 		(fields_autoplaced yes)
-		(property "Reference" "L3"
+		(property "Reference" "L4"
 			(at 181.61 62.23 90)
 			(show_name no)
@@
 			(project "WINLAB-LP-Radio-Sensor-Hub"
 				(path "/0de7ee4a-bb98-4bc6-bb89-3afafc4b94b5/415caeb0-0f13-4c6e-8f8f-fa1df5ea5ac9"
-					(reference "L3")
+					(reference "L4")
 					(unit 1)
 				)
@@
 		(dnp no)
 		(fields_autoplaced yes)
-		(property "Reference" "U4"
+		(property "Reference" "U6"
 			(at 102.87 72.3198 0)
 			(show_name no)
@@
 			(project "WINLAB-LP-Radio-Sensor-Hub"
 				(path "/0de7ee4a-bb98-4bc6-bb89-3afafc4b94b5/415caeb0-0f13-4c6e-8f8f-fa1df5ea5ac9"
-					(reference "U4")
-					(unit 1)
-				)
+					(reference "U6")
+					(unit 1)
+				)
