File: RF.kicad_sch (KiCad schematic)
At the start: 12 parts, among them J2 Conn_Coaxial, J3 Conn_Coaxial, U6 ADG902BRMZ

Commit message: completed layout and routing with preliminary matching network
Parts:
- renumbered C22 to C26, C23 to C27, C24 to C28, C25 to C29, C26 to C30, J2 to J4, J3 to J5, U6 to U7
Changed lines of the file:
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@@
 		(dnp no)
 		(fields_autoplaced yes)
-		(property "Reference" "#PWR024"
+		(property "Reference" "#PWR034"
 			(at 240.03 78.74 0)
 			(hide yes)
@@
 			(project "WINLAB-LP-Radio-Sensor-Hub"
 				(path "/0de7ee4a-bb98-4bc6-bb89-3afafc4b94b5/415caeb0-0f13-4c6e-8f8f-fa1df5ea5ac9"
-					(reference "#PWR024")
+					(reference "#PWR034")
 					(unit 1)
 				)
@@
 		(dnp no)
 		(fields_autoplaced yes)
-		(property "Reference" "J2"
+		(property "Reference" "J4"
 			(at 116.84 77.7631 0)
 			(show_name no)
@@
 			(project "WINLAB-LP-Radio-Sensor-Hub"
 				(path "/0de7ee4a-bb98-4bc6-bb89-3afafc4b94b5/415caeb0-0f13-4c6e-8f8f-fa1df5ea5ac9"
-					(reference "J2")
+					(reference "J4")
 					(unit 1)
 				)
@@
 		(dnp no)
 		(fields_autoplaced yes)
-		(property "Reference" "C24"
+		(property "Reference" "C28"
 			(at 194.31 69.8499 0)
 			(show_name no)
@@
 			(project "WINLAB-LP-Radio-Sensor-Hub"
 				(path "/0de7ee4a-bb98-4bc6-bb89-3afafc4b94b5/415caeb0-0f13-4c6e-8f8f-fa1df5ea5ac9"
-					(reference "C24")
+					(reference "C28")
 					(unit 1)
 				)
@@
 		(dnp no)
 		(fields_autoplaced yes)
-		(property "Reference" "C25"
+		(property "Reference" "C29"
 			(at 212.09 69.8499 0)
 			(show_name no)
@@
 			(project "WINLAB-LP-Radio-Sensor-Hub"
 				(path "/0de7ee4a-bb98-4bc6-bb89-3afafc4b94b5/415caeb0-0f13-4c6e-8f8f-fa1df5ea5ac9"
-					(reference "C25")
+					(reference "C29")
 					(unit 1)
 				)
@@
 		(dnp no)
 		(fields_autoplaced yes)
-		(property "Reference" "C23"
+		(property "Reference" "C27"
 			(at 168.91 49.53 90)
 			(show_name no)
@@
 			(project "WINLAB-LP-Radio-Sensor-Hub"
 				(path "/0de7ee4a-bb98-4bc6-bb89-3afafc4b94b5/415caeb0-0f13-4c6e-8f8f-fa1df5ea5ac9"
-					(reference "C23")
+					(reference "C27")
 					(unit 1)
 				)
@@
 		(dnp no)
 		(fields_autoplaced yes)
-		(property "Reference" "#PWR023"
+		(property "Reference" "#PWR033"
 			(at 208.28 81.28 0)
 			(hide yes)
@@
 			(project "WINLAB-LP-Radio-Sensor-Hub"
 				(path "/0de7ee4a-bb98-4bc6-bb89-3afafc4b94b5/415caeb0-0f13-4c6e-8f8f-fa1df5ea5ac9"
-					(reference "#PWR023")
+					(reference "#PWR033")
 					(unit 1)
 				)
@@
 		(dnp no)
 		(fields_autoplaced yes)
-		(property "Reference" "C22"
+		(property "Reference" "C26"
 			(at 95.25 57.1499 0)
 			(show_name no)
@@
 			(project "WINLAB-LP-Radio-Sensor-Hub"
 				(path "/0de7ee4a-bb98-4bc6-bb89-3afafc4b94b5/415caeb0-0f13-4c6e-8f8f-fa1df5ea5ac9"
-					(reference "C22")
+					(reference "C26")
 					(unit 1)
 				)
@@
 		(dnp no)
 		(fields_autoplaced yes)
-		(property "Reference" "#PWR020"
+		(property "Reference" "#PWR030"
 			(at 91.44 58.42 0)
 			(hide yes)
@@
 			(project "WINLAB-LP-Radio-Sensor-Hub"
 				(path "/0de7ee4a-bb98-4bc6-bb89-3afafc4b94b5/415caeb0-0f13-4c6e-8f8f-fa1df5ea5ac9"
-					(reference "#PWR020")
+					(reference "#PWR030")
 					(unit 1)
 				)
@@
 		(dnp no)
 		(fields_autoplaced yes)
-		(property "Reference" "C26"
+		(property "Reference" "C30"
 			(at 223.52 59.69 90)
 			(show_name no)
@@
 			(project "WINLAB-LP-Radio-Sensor-Hub"
 				(path "/0de7ee4a-bb98-4bc6-bb89-3afafc4b94b5/415caeb0-0f13-4c6e-8f8f-fa1df5ea5ac9"
-					(reference "C26")
+					(reference "C30")
 					(unit 1)
 				)
@@
 		(dnp no)
 		(fields_autoplaced yes)
-		(property "Reference" "#PWR019"
+		(property "Reference" "#PWR029"
 			(at 85.09 102.87 0)
 			(hide yes)
@@
 			(project "WINLAB-LP-Radio-Sensor-Hub"
 				(path "/0de7ee4a-bb98-4bc6-bb89-3afafc4b94b5/415caeb0-0f13-4c6e-8f8f-fa1df5ea5ac9"
-					(reference "#PWR019")
+					(reference "#PWR029")
 					(unit 1)
 				)
@@
 		(dnp no)
 		(fields_autoplaced yes)
-		(property "Reference" "J3"
+		(property "Reference" "J5"
 			(at 243.84 66.3331 0)
 			(show_name no)
@@
 			(project "WINLAB-LP-Radio-Sensor-Hub"
 				(path "/0de7ee4a-bb98-4bc6-bb89-3afafc4b94b5/415caeb0-0f13-4c6e-8f8f-fa1df5ea5ac9"
-					(reference "J3")
+					(reference "J5")
 					(unit 1)
 				)
@@
 		(dnp no)
 		(fields_autoplaced yes)
-		(property "Reference" "#PWR021"
+		(property "Reference" "#PWR031"
 			(at 91.44 68.58 0)
 			(hide yes)
@@
 			(project "WINLAB-LP-Radio-Sensor-Hub"
 				(path "/0de7ee4a-bb98-4bc6-bb89-3afafc4b94b5/415caeb0-0f13-4c6e-8f8f-fa1df5ea5ac9"
-					(reference "#PWR021")
+					(reference "#PWR031")
 					(unit 1)
 				)
@@
 		(dnp no)
 		(fields_autoplaced yes)
-		(property "Reference" "U6"
+		(property "Reference" "U7"
 			(at 102.87 72.3198 0)
 			(show_name no)
@@
 			(project "WINLAB-LP-Radio-Sensor-Hub"
 				(path "/0de7ee4a-bb98-4bc6-bb89-3afafc4b94b5/415caeb0-0f13-4c6e-8f8f-fa1df5ea5ac9"
-					(reference "U6")
+					(reference "U7")
 					(unit 1)
 				)
@@
 		(dnp no)
 		(fields_autoplaced yes)
-		(property "Reference" "#PWR022"
+		(property "Reference" "#PWR032"
 			(at 190.5 81.28 0)
 			(hide yes)
@@
 			(project "WINLAB-LP-Radio-Sensor-Hub"
 				(path "/0de7ee4a-bb98-4bc6-bb89-3afafc4b94b5/415caeb0-0f13-4c6e-8f8f-fa1df5ea5ac9"
-					(reference "#PWR022")
-					(unit 1)
-				)
+					(reference "#PWR032")
+					(unit 1)
+				)

Commit message: switch to 0402 matching network closer to reference design
Parts:
- C27, C28, C29, C30: footprint Capacitor_SMD:C_0603_1608Metric_Pad1.08x0.95mm_HandSolder -> Capacitor_SMD:C_0402_1005Metric
- L2, L3, L4, L5: footprint Inductor_SMD:L_0603_1608Metric_Pad1.05x0.95mm_HandSolder -> Inductor_SMD:L_0402_1005Metric
Changed lines of the file:
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@@
 			)
 		)
-		(property "Footprint" "Inductor_SMD:L_0603_1608Metric_Pad1.05x0.95mm_HandSolder"
+		(property "Footprint" "Inductor_SMD:L_0402_1005Metric"
 			(at 168.91 82.55 0)
 			(hide yes)
@@
 			)
 		)
-		(property "Footprint" "Capacitor_SMD:C_0603_1608Metric_Pad1.08x0.95mm_HandSolder"
+		(property "Footprint" "Capacitor_SMD:C_0402_1005Metric"
 			(at 189.5348 74.93 0)
 			(hide yes)
@@
 			)
 		)
-		(property "Footprint" "Capacitor_SMD:C_0603_1608Metric_Pad1.08x0.95mm_HandSolder"
+		(property "Footprint" "Capacitor_SMD:C_0402_1005Metric"
 			(at 207.3148 74.93 0)
 			(hide yes)
@@
 			)
 		)
-		(property "Footprint" "Capacitor_SMD:C_0603_1608Metric_Pad1.08x0.95mm_HandSolder"
+		(property "Footprint" "Capacitor_SMD:C_0402_1005Metric"
 			(at 172.72 58.1152 0)
 			(hide yes)
@@
 			)
 		)
-		(property "Footprint" "Inductor_SMD:L_0603_1608Metric_Pad1.05x0.95mm_HandSolder"
+		(property "Footprint" "Inductor_SMD:L_0402_1005Metric"
 			(at 199.39 67.31 0)
 			(hide yes)
@@
 			)
 		)
-		(property "Footprint" "Capacitor_SMD:C_0603_1608Metric_Pad1.08x0.95mm_HandSolder"
+		(property "Footprint" "Capacitor_SMD:C_0402_1005Metric"
 			(at 227.33 68.2752 0)
 			(hide yes)
@@
 			)
 		)
-		(property "Footprint" "Inductor_SMD:L_0603_1608Metric_Pad1.05x0.95mm_HandSolder"
+		(property "Footprint" "Inductor_SMD:L_0402_1005Metric"
 			(at 168.91 67.31 0)
 			(hide yes)
@@
 			)
 		)
-		(property "Footprint" "Inductor_SMD:L_0603_1608Metric_Pad1.05x0.95mm_HandSolder"
+		(property "Footprint" "Inductor_SMD:L_0402_1005Metric"
 			(at 181.61 67.31 0)
 			(hide yes)

Commit message: add LCSC part number properties in preparation for JLCPCB assembly order
Parts:
- C26: LCSC Part Number (none) -> C14663
- C27: LCSC Part Number (none) -> C161314
- C28: LCSC Part Number (none) -> C2220960
- C29: LCSC Part Number (none) -> C161309
- C30: LCSC Part Number (none) -> C71693
- J4, J5: LCSC Part Number (none) -> C7542042
- L2: LCSC Part Number (none) -> C3911137
- L3: LCSC Part Number (none) -> C91622
- L4: LCSC Part Number (none) -> C3910751
- L5: LCSC Part Number (none) -> C341684
- U7: LCSC Part Number (none) -> C207407
