File: MCU.kicad_sch (KiCad schematic)
At the start: 35 parts, among them J1 FTSH-105-01-L-DV-K-A, U1 EFR32FG23L020F128GM40-C, U2 Si7021-A20, Y1 39MHz 10pF

Commit message: more layout and routing work
Connections:
- net DBG_UART_RX is gone; now on net VCOM_RX: J1.4
- net DBG_UART_TX is gone; now on net VCOM_TX: J1.5
- net BTN_USR: now also S2.3 (NO_1), S2.4 (NO_2); no longer S2.1 (COM_1), S2.2 (COM_2)
- net RESET: now also S1.3 (NO_1), S1.4 (NO_2); no longer S1.1 (COM_1), S1.2 (COM_2)
- new net: R4.1, S2.1 (COM_1), S2.2 (COM_2)
- new net: R2.1, S1.1 (COM_1), S1.2 (COM_2)
Changed lines of the file:
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@@
 	)
 	(junction
-		(at 148.59 142.24)
-		(diameter 0)
-		(color 0 0 0 0)
-	)
-	(junction
 		(at 194.31 86.36)
 		(diameter 0)
@@
 	)
 	(junction
+		(at 148.59 142.24)
+		(diameter 0)
+		(color 0 0 0 0)
+	)
+	(junction
 		(at 207.01 63.5)
 		(diameter 0)
@@
 	)
 	(junction
-		(at 27.94 57.15)
+		(at 59.69 139.7)
 		(diameter 0)
 		(color 0 0 0 0)
 	)
 	(junction
-		(at 59.69 137.16)
+		(at 27.94 57.15)
 		(diameter 0)
 		(color 0 0 0 0)
 	)
 	(junction
-		(at 44.45 77.47)
+		(at 59.69 137.16)
 		(diameter 0)
 		(color 0 0 0 0)
 	)
 	(junction
-		(at 59.69 139.7)
+		(at 44.45 77.47)
 		(diameter 0)
 		(color 0 0 0 0)
@@
 	(wire
 		(pts
+			(xy 148.59 142.24) (xy 179.07 142.24)
+		)
+		(stroke
+			(width 0)
+			(type default)
+		)
+	)
+	(wire
+		(pts
 			(xy 144.78 166.37) (xy 144.78 172.72)
 		)
@@
 	(wire
 		(pts
-			(xy 59.69 139.7) (xy 90.17 139.7)
-		)
-		(stroke
-			(width 0)
-			(type default)
-		)
-	)
-	(wire
-		(pts
 			(xy 106.68 44.45) (xy 88.9 44.45)
 		)
@@
 	(wire
 		(pts
-			(xy 148.59 142.24) (xy 179.07 142.24)
-		)
-		(stroke
-			(width 0)
-			(type default)
-		)
-	)
-	(wire
-		(pts
 			(xy 189.23 63.5) (xy 194.31 63.5)
 		)
@@
 	(wire
 		(pts
+			(xy 59.69 139.7) (xy 90.17 139.7)
+		)
+		(stroke
+			(width 0)
+			(type default)
+		)
+	)
+	(wire
+		(pts
 			(xy 44.45 85.09) (xy 57.15 85.09)
 		)
@@
 		)
 	)
-	(global_label "DBG_UART_TX"
+	(global_label "VCOM_TX"
 		(shape input)
 		(at 252.73 142.24 0)
@@
 		)
 		(property "Intersheetrefs" "${INTERSHEET_REFS}"
-			(at 268.2942 142.24 0)
+			(at 264.0004 142.24 0)
 			(hide yes)
 			(show_name no)
@@
 		)
 	)
-	(global_label "DBG_UART_RX"
+	(global_label "VCOM_RX"
 		(shape output)
 		(at 229.87 144.78 180)
@@
 		)
 		(property "Intersheetrefs" "${INTERSHEET_REFS}"
-			(at 214.0034 144.78 0)
+			(at 218.2972 144.78 0)
 			(hide yes)
 			(show_name no)
@@
 	(symbol
 		(lib_id "SamacSys_Parts:RKB2SJM250SMTR_LFS")
-		(at 148.59 139.7 0)
+		(at 148.59 142.24 0)
+		(mirror x)
 		(unit 1)
 		(body_style 1)
@@
 		(in_pos_files yes)
 		(dnp no)
-		(fields_autoplaced yes)
 		(property "Reference" "S2"
-			(at 163.83 132.08 0)
+			(at 163.83 149.86 0)
 			(show_name no)
 			(do_not_autoplace no)
@@
 		)
 		(property "Value" "RKB2SJM250SMTR_LFS"
-			(at 163.83 134.62 0)
+			(at 163.83 147.32 0)
 			(show_name no)
 			(do_not_autoplace no)
@@
 		)
 		(property "Footprint" "RKB2SJM250SMTRLFS"
-			(at 175.26 234.62 0)
+			(at 175.26 47.32 0)
 			(hide yes)
 			(show_name no)
@@
 		)
 		(property "Datasheet" "https://www.ckswitches.com/media/3130/ck_rk_datasheet.pdf"
-			(at 175.26 334.62 0)
+			(at 175.26 -52.68 0)
 			(hide yes)
 			(show_name no)
@@
 		)
 		(property "Description" "Tactile Switches J Bend SMT Term 180gf Force"
-			(at 148.59 139.7 0)
+			(at 148.59 142.24 0)
 			(hide yes)
 			(show_name no)
@@
 		)
 		(property "Height" "2.7"
-			(at 175.26 534.62 0)
+			(at 175.26 -252.68 0)
 			(hide yes)
 			(show_name no)
@@
 		)
 		(property "Mouser Part Number" "611-RKB2SJM250SMTRLF"
-			(at 175.26 634.62 0)
+			(at 175.26 -352.68 0)
 			(hide yes)
 			(show_name no)
@@
 		)
 		(property "Mouser Price/Stock" "https://www.mouser.co.uk/ProductDetail/CK/RKB2SJM250SMTR-LFS?qs=iLbezkQI%252Bsj518EgFgehgw%3D%3D"
-			(at 175.26 734.62 0)
+			(at 175.26 -452.68 0)
 			(hide yes)
 			(show_name no)
@@
 		)
 		(property "Manufacturer_Name" "C & K COMPONENTS"
-			(at 175.26 834.62 0)
+			(at 175.26 -552.68 0)
 			(hide yes)
 			(show_name no)
@@
 		)
 		(property "Manufacturer_Part_Number" "RKB2SJM250SMTR LFS"
-			(at 175.26 934.62 0)
+			(at 175.26 -652.68 0)
 			(hide yes)
 			(show_name no)
@@
 	(symbol
 		(lib_id "SamacSys_Parts:RKB2SJM250SMTR_LFS")
-		(at 59.69 137.16 0)
+		(at 59.69 139.7 0)
+		(mirror x)
 		(unit 1)
 		(body_style 1)
@@
 		(in_pos_files yes)
 		(dnp no)
-		(fields_autoplaced yes)
 		(property "Reference" "S1"
-			(at 74.93 129.54 0)
+			(at 74.93 147.32 0)
 			(show_name no)
 			(do_not_autoplace no)
@@
 		)
 		(property "Value" "RKB2SJM250SMTR_LFS"
-			(at 74.93 132.08 0)
+			(at 74.93 144.78 0)
 			(show_name no)
 			(do_not_autoplace no)
@@
 		)
 		(property "Footprint" "RKB2SJM250SMTRLFS"
-			(at 86.36 232.08 0)
+			(at 86.36 44.78 0)
 			(hide yes)
 			(show_name no)
@@
 		)
 		(property "Datasheet" "https://www.ckswitches.com/media/3130/ck_rk_datasheet.pdf"
-			(at 86.36 332.08 0)
+			(at 86.36 -55.22 0)
 			(hide yes)
 			(show_name no)
@@
 		)
 		(property "Description" "Tactile Switches J Bend SMT Term 180gf Force"
-			(at 59.69 137.16 0)
+			(at 59.69 139.7 0)
 			(hide yes)
 			(show_name no)
@@
 		)
 		(property "Height" "2.7"
-			(at 86.36 532.08 0)
+			(at 86.36 -255.22 0)
 			(hide yes)
 			(show_name no)
@@
 		)
 		(property "Mouser Part Number" "611-RKB2SJM250SMTRLF"
-			(at 86.36 632.08 0)
+			(at 86.36 -355.22 0)
 			(hide yes)
 			(show_name no)
@@
 		)
 		(property "Mouser Price/Stock" "https://www.mouser.co.uk/ProductDetail/CK/RKB2SJM250SMTR-LFS?qs=iLbezkQI%252Bsj518EgFgehgw%3D%3D"
-			(at 86.36 732.08 0)
+			(at 86.36 -455.22 0)
 			(hide yes)
 			(show_name no)
@@
 		)
 		(property "Manufacturer_Name" "C & K COMPONENTS"
-			(at 86.36 832.08 0)
+			(at 86.36 -555.22 0)
 			(hide yes)
 			(show_name no)
@@
 		)
 		(property "Manufacturer_Part_Number" "RKB2SJM250SMTR LFS"
-			(at 86.36 932.08 0)
+			(at 86.36 -655.22 0)
 			(hide yes)
 			(show_name no)
