File: MCU.kicad_sch (KiCad schematic)
At the start: 36 parts, among them J1 FTSH-105-01-L-DV-K-A, U1 EFR32FG23L020F128GM40-C, U2 Si7021-A20, Y1 39MHz 10pF

Commit message: layout and silkscreen tweaks
Parts:
- FB1: value FerriteBead -> BLM18SG700TZ1D
- FB2, FB3: value FerriteBead -> 0R
- FB4: value FerriteBead -> BLM18PG330SN1D
Changed lines of the file:
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@@
 			)
 		)
-		(property "Value" "FerriteBead"
+		(property "Value" "0R"
 			(at 83.7692 72.39 90)
 			(show_name no)
@@
 			)
 		)
-		(property "Value" "FerriteBead"
+		(property "Value" "BLM18PG330SN1D"
 			(at 118.1608 72.39 90)
 			(show_name no)
@@
 			)
 		)
-		(property "Value" "FerriteBead"
+		(property "Value" "0R"
 			(at 118.0592 52.07 90)
 			(show_name no)
@@
 			)
 		)
-		(property "Value" "FerriteBead"
+		(property "Value" "BLM18SG700TZ1D"
 			(at 83.7692 52.07 90)
 			(show_name no)

Commit message: change CN3063 input diode and tie temp to ground, HW UVP LPF, change DCDC input capacitance setup, remove crystal loading caps, add series resistors on CH340 serial lines, add via fence on CPWGs
Parts:
- removed C6, C7: 12p, Capacitor_SMD:C_0603_1608Metric_Pad1.08x0.95mm_HandSolder, symbol Device:C
- C19: value 1u -> 10u
Changed lines of the file:
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@@
 	)
 	(junction
-		(at 137.16 24.13)
-		(diameter 0)
-		(color 0 0 0 0)
-	)
-	(junction
 		(at 193.04 101.6)
 		(diameter 0)
@@
 	)
 	(junction
-		(at 157.48 33.02)
-		(diameter 0)
-		(color 0 0 0 0)
-	)
-	(junction
 		(at 39.37 147.32)
 		(diameter 0)
@@
 	)
 	(junction
-		(at 137.16 33.02)
-		(diameter 0)
-		(color 0 0 0 0)
-	)
-	(junction
 		(at 148.59 142.24)
 		(diameter 0)
@@
 	)
 	(junction
-		(at 147.32 24.13)
-		(diameter 0)
-		(color 0 0 0 0)
-	)
-	(junction
 		(at 142.24 187.96)
 		(diameter 0)
@@
 	(wire
 		(pts
-			(xy 147.32 24.13) (xy 137.16 24.13)
+			(xy 132.08 26.67) (xy 147.32 26.67)
 		)
 		(stroke
@@
 	(wire
 		(pts
-			(xy 137.16 24.13) (xy 120.65 24.13)
-		)
-		(stroke
-			(width 0)
-			(type default)
-		)
-	)
-	(wire
-		(pts
 			(xy 39.37 148.59) (xy 39.37 147.32)
 		)
@@
 	(wire
 		(pts
-			(xy 147.32 27.94) (xy 147.32 24.13)
+			(xy 147.32 26.67) (xy 147.32 27.94)
 		)
 		(stroke
@@
 	(wire
 		(pts
-			(xy 157.48 25.4) (xy 157.48 24.13)
-		)
-		(stroke
-			(width 0)
-			(type default)
-		)
-	)
-	(wire
-		(pts
 			(xy 60.96 175.26) (xy 62.23 175.26)
 		)
@@
 	(wire
 		(pts
-			(xy 137.16 24.13) (xy 137.16 25.4)
-		)
-		(stroke
-			(width 0)
-			(type default)
-		)
-	)
-	(wire
-		(pts
-			(xy 157.48 24.13) (xy 147.32 24.13)
-		)
-		(stroke
-			(width 0)
-			(type default)
-		)
-	)
-	(wire
-		(pts
 			(xy 237.49 72.39) (xy 237.49 63.5)
 		)
@@
 			)
 		)
-		(property "Value" "1u"
+		(property "Value" "10u"
 			(at 259.08 91.4399 0)
 			(show_name no)
@@
 	(symbol
 		(lib_id "power:GND")
-		(at 120.65 24.13 0)
+		(at 132.08 26.67 0)
 		(unit 1)
 		(body_style 1)
@@
 		(fields_autoplaced yes)
 		(property "Reference" "#PWR06"
-			(at 120.65 30.48 0)
+			(at 132.08 33.02 0)
 			(hide yes)
 			(show_name no)
@@
 		)
 		(property "Value" "GND"
-			(at 120.65 29.21 0)
+			(at 132.08 31.75 0)
 			(show_name no)
 			(do_not_autoplace no)
@@
 		)
 		(property "Footprint" ""
-			(at 120.65 24.13 0)
+			(at 132.08 26.67 0)
 			(hide yes)
 			(show_name no)
@@
 		)
 		(property "Datasheet" ""
-			(at 120.65 24.13 0)
+			(at 132.08 26.67 0)
 			(hide yes)
 			(show_name no)
@@
 		)
 		(property "Description" "Power symbol creates a global label with name \"GND\" , ground"
-			(at 120.65 24.13 0)
+			(at 132.08 26.67 0)
 			(hide yes)
 			(show_name no)
@@
 					(unit 1)
 				)
-			)
-		)
-	)
-	(symbol
-		(lib_id "Device:C")
-		(at 157.48 29.21 0)
-		(mirror y)
-		(unit 1)
-		(body_style 1)
-		(exclude_from_sim no)
-		(in_bom yes)
-		(on_board yes)
-		(in_pos_files yes)
-		(dnp no)
-		(property "Reference" "C7"
-			(at 161.29 27.9399 0)
-			(show_name no)
-			(do_not_autoplace no)
-			(effects
-				(font
-					(size 1.27 1.27)
-				)
-				(justify right)
-			)
-		)
-		(property "Value" "12p"
-			(at 161.29 30.4799 0)
-			(show_name no)
-			(do_not_autoplace no)
-			(effects
-				(font
-					(size 1.27 1.27)
-				)
-				(justify right)
-			)
-		)
-		(property "Footprint" "Capacitor_SMD:C_0603_1608Metric_Pad1.08x0.95mm_HandSolder"
-			(at 156.5148 33.02 0)
-			(hide yes)
-			(show_name no)
-			(do_not_autoplace no)
-			(effects
-				(font
-					(size 1.27 1.27)
-				)
-			)
-		)
-		(property "Datasheet" ""
-			(at 157.48 29.21 0)
-			(hide yes)
-			(show_name no)
-			(do_not_autoplace no)
-			(effects
-				(font
-					(size 1.27 1.27)
-				)
-			)
-		)
-		(property "Description" "Unpolarized capacitor"
-			(at 157.48 29.21 0)
-			(hide yes)
-			(show_name no)
-			(do_not_autoplace no)
-			(effects
-				(font
-					(size 1.27 1.27)
-				)
-			)
-		)
-		(pin "1"
-		)
-		(pin "2"
-		)
-		(instances
-			(project "WINLAB-LP-Radio-Sensor-Hub"
-				(path "/0de7ee4a-bb98-4bc6-bb89-3afafc4b94b5/f02c211f-c559-4db5-8225-ca108efc3892"
-					(reference "C7")
-					(unit 1)
-				)
-			)
-		)
-	)
-	(symbol
-		(lib_id "Device:C")
-		(at 137.16 29.21 0)
-		(unit 1)
-		(body_style 1)
-		(exclude_from_sim no)
-		(in_bom yes)
-		(on_board yes)
-		(in_pos_files yes)
-		(dnp no)
-		(property "Reference" "C6"
-			(at 133.35 27.9399 0)
-			(show_name no)
-			(do_not_autoplace no)
-			(effects
-				(font
-					(size 1.27 1.27)
-				)
-				(justify right)
-			)
-		)
-		(property "Value" "12p"
-			(at 133.35 30.4799 0)
-			(show_name no)
-			(do_not_autoplace no)
-			(effects
-				(font
-					(size 1.27 1.27)
-				)
-				(justify right)
-			)
-		)
-		(property "Footprint" "Capacitor_SMD:C_0603_1608Metric_Pad1.08x0.95mm_HandSolder"
-			(at 138.1252 33.02 0)
-			(hide yes)
-			(show_name no)
-			(do_not_autoplace no)
-			(effects
-				(font
-					(size 1.27 1.27)
-				)
-			)
-		)
-		(property "Datasheet" ""
-			(at 137.16 29.21 0)
-			(hide yes)
-			(show_name no)
-			(do_not_autoplace no)
-			(effects
-				(font
-					(size 1.27 1.27)
-				)
-			)
-		)
-		(property "Description" "Unpolarized capacitor"
-			(at 137.16 29.21 0)
-			(hide yes)
-			(show_name no)
-			(do_not_autoplace no)
-			(effects
-				(font
-					(size 1.27 1.27)
-				)
-			)
-		)
-		(pin "1"
-		)
-		(pin "2"
-		)
-		(instances
-			(project "WINLAB-LP-Radio-Sensor-Hub"
-				(path "/0de7ee4a-bb98-4bc6-bb89-3afafc4b94b5/f02c211f-c559-4db5-8225-ca108efc3892"
-					(reference "C6")
-					(unit 1)
-				)

Commit message: add LCSC part number properties in preparation for JLCPCB assembly order
Parts:
- C1, C11, C13, C14, C15, C16, C8, C9: LCSC Part Number (none) -> C14663
- C10, C17, C18, C2: LCSC Part Number (none) -> C15849
- C12: LCSC Part Number (none) -> C1779
- C19: LCSC Part Number (none) -> C19702
- C3: LCSC Part Number (none) -> C1623
- C4, C5: LCSC Part Number (none) -> C14858
- FB1: LCSC Part Number (none) -> C882974
- FB2, FB3: LCSC Part Number (none) -> C21189
- FB4: LCSC Part Number (none) -> C88984
- J1: LCSC Part Number (none) -> C21318670
- L1: LCSC Part Number (none) -> C6364793
- R1: LCSC Part Number (none) -> C23179
- R2, R4: LCSC Part Number (none) -> C22775
- R3: LCSC Part Number (none) -> C25804
- S1, S2: LCSC Part Number (none) -> C2927789
- Y1: LCSC Part Number (none) -> C51949557
